File: kicad_files/lc709203f.kicad_sch (KiCad schematic)
At the start: 0 parts

Commit message: Completed fuel gauge schematic based on application guidance provided in the LC709203F datasheet.
Parts:
- added C1: 0.1uF, symbol Device:C
- added R1, R2, R3, R5: 10000, symbol Device:R
- added R4: 100, symbol Device:R
- added TH1: 10000, symbol Device:Thermistor_NTC
- added U1: LC709203FQH-01TWG, Package_DFN_QFN:WDFN-8-1EP_4x3mm_P0.65mm_EP2.4x1.8mm, symbol Battery_Management:LC709203FQH-01TWG
Connections:
- new net: R3.2, R4.1, TH1.1
- new net: R4.2, U1.6 (T_{SENSE})
- new net: R5.2, U1.4 (~{ALARMB})
- new net: R3.1, U1.5 (T_{SW})
- new net: R2.2, U1.7 (SDA)
- new net: R1.2, U1.8 (SCL)
- new net Bat+: C1.1, U1.3 (V_{DD})
- new net GNDPWR: C1.2, TH1.2, U1.1 (TEST), U1.2 (V_{SS})
- new net VDD (from 3.3V rail): R1.1, R2.1, R5.1
